File: hardware/chase.sch (KiCad schematic (older format))
At the start: 51 parts, among them J1 THD0509-04CL-GF, Q1 DMC3400SDW-7, Q2 DMN61D9UDW, Q3 DMN61D9UDW, SW1 TS-1187A-B-A-B, T1 TestPoint, T2 TestPoint, T3 TestPoint, T4 TestPoint, T5 TestPoint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

Commit message: Replace J1 with 6 pin connector, use cheaper resistor for 430 ohms.
Parts:
- J1: value THD0509-04CL-GF -> FH12-6S-0.5SH(55); footprint chase-libs:THD050904CLGF -> Connector_FFC-FPC:Hirose_FH12-6S-0.5SH_1x06-1MP_P0.50mm_Horizontal; symbol Connector:Conn_01x04_Female -> Connector:Conn_01x06_Female; Description FPC Contact,Top and Bottom 4 0.020\"（0.50mm） SMD,P=0.5mm FF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 -> FPC Contact 6pin SMD horizontal; MPN THD0509-04CL-GF -> FH12-6S-0.5SH(55)
- R2, R70, R71, R72: MPN ARG02FTC4300 -> 0402WGF4300TCE; description 430 ±1% 1/16W 0402 High Precision & Low TCR SMD Resistors R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 -> thick film; SMD; 0402; 430Ω; 63mW; ±1%; -55÷155°C
Connections:
- net D+: now also J1.2 (Pin_2), U1.7 (PB2); no longer U1.2 (XTAL1/PB3)
- net D-: now also U1.5 (AREF/PB0); no longer U1.3 (XTAL2/PB4)
- net GND: now also J1.5 (Pin_5); no longer J1.4 (Pin_4)
- net LED Driver 1/RCK: now also U1.3 (XTAL2/PB4); no longer U1.7 (PB2)
- net LED Driver 1/SRCK: now also U1.2 (XTAL1/PB3); no longer U1.5 (AREF/PB0)
- net VBUS: now also J1.4 (Pin_4); no longer J1.3 (Pin_3)
- net XVCC: now also J1.3 (Pin_3); no longer J1.2 (Pin_2)
- no-connect marks 12 -> 13
Other:
- note added: "When there is USB power, \nXVCC is grounded."
- note added: "XSIG1 and XSIG2 are intended for\nconnecting a microphone, buzzer\nor EEPROM or other addon boards."
- note removed: "ADC1 point is intended for\nconnecting a microphone\nor other input to the ATtiny."
- note removed: "When there is USB power, \nADC1 is disconnected."
Changed lines of the file:
@@
 encoding utf-8
 Sheet 1 6
-Title "3.3V LED CHASER with USB-C and LiPo - 60 LEDS"
-Date "2020-02-11"
-Rev "8"
-Comp "https://github.com/krk"
+Title "3.3V/5V LED CHASER with USB-C and LiPo - 60 LEDS"
+Date "2020-02-20"
+Rev "9"
+Comp "https://github.com/krk/chase-badge"
 Comment1 ""
 Comment2 ""
@@
 F 1 "430" V 3034 4100 50  0000 C CNN
 F 2 "Resistor_SMD:R_0402_1005Metric" V 3080 4100 50  0001 C CNN
-F 3 "https://datasheet.lcsc.com/szlcsc/1912111437_Viking-Tech-ARG02FTC4300_C284568.pdf" H 3150 4100 50  0001 C CNN
-F 4 "430 ±1% 1/16W 0402 High Precision & Low TCR SMD Resistors RoHS" V 3150 4100 50  0001 C CNN "description"
-F 5 "ARG02FTC4300" V 3150 4100 50  0001 C CNN "MPN"
+F 3 "https://www.tme.eu/Document/9e42ba54d36a9bd3dfa2901986ac022d/rezystor-smd.pdf" H 3150 4100 50  0001 C CNN
+F 4 "thick film; SMD; 0402; 430Ω; 63mW; ±1%; -55÷155°C" V 3150 4100 50  0001 C CNN "description"
+F 5 "0402WGF4300TCE" V 3150 4100 50  0001 C CNN "MPN"
 	1    3150 4100
 	0    1    1    0
@@
 F 1 "430" V 3034 4450 50  0000 C CNN
 F 2 "Resistor_SMD:R_0402_1005Metric" V 3080 4450 50  0001 C CNN
-F 3 "https://datasheet.lcsc.com/szlcsc/1912111437_Viking-Tech-ARG02FTC4300_C284568.pdf" H 3150 4450 50  0001 C CNN
-F 4 "430 ±1% 1/16W 0402 High Precision & Low TCR SMD Resistors RoHS" V 3150 4450 50  0001 C CNN "description"
-F 5 "ARG02FTC4300" V 3150 4450 50  0001 C CNN "MPN"
+F 3 "https://www.tme.eu/Document/9e42ba54d36a9bd3dfa2901986ac022d/rezystor-smd.pdf" H 3150 4450 50  0001 C CNN
+F 4 "thick film; SMD; 0402; 430Ω; 63mW; ±1%; -55÷155°C" V 3150 4450 50  0001 C CNN "description"
+F 5 "0402WGF4300TCE" V 3150 4450 50  0001 C CNN "MPN"
 	1    3150 4450
 	0    1    1    0
@@
 F 1 "430" V 3034 4800 50  0000 C CNN
 F 2 "Resistor_SMD:R_0402_1005Metric" V 3080 4800 50  0001 C CNN
-F 3 "https://datasheet.lcsc.com/szlcsc/1912111437_Viking-Tech-ARG02FTC4300_C284568.pdf" H 3150 4800 50  0001 C CNN
-F 4 "430 ±1% 1/16W 0402 High Precision & Low TCR SMD Resistors RoHS" V 3150 4800 50  0001 C CNN "description"
-F 5 "ARG02FTC4300" V 3150 4800 50  0001 C CNN "MPN"
+F 3 "https://www.tme.eu/Document/9e42ba54d36a9bd3dfa2901986ac022d/rezystor-smd.pdf" H 3150 4800 50  0001 C CNN
+F 4 "thick film; SMD; 0402; 430Ω; 63mW; ±1%; -55÷155°C" V 3150 4800 50  0001 C CNN "description"
+F 5 "0402WGF4300TCE" V 3150 4800 50  0001 C CNN "MPN"
 	1    3150 4800
 	0    1    1    0
@@
 Wire Wire Line
 	3800 1200 3800 1500
-Wire Wire Line
-	9850 1450 9850 1250
-Connection ~ 9850 1450
-Wire Wire Line
-	8100 1650 8200 1650
-Wire Wire Line
-	9800 1450 9800 1550
-Connection ~ 9800 1550
 Text GLabel 2700 5450 2    50   Input ~ 0
 D+
@@
 Text GLabel 2700 5750 2    50   Input ~ 0
 D-
-Text GLabel 8200 700  0    50   Input ~ 0
-D+
-Text GLabel 8200 850  0    50   Input ~ 0
+Text GLabel 8200 650  0    50   Input ~ 0
 D-
 Wire Wire Line
-	8200 700  8400 700
-Wire Wire Line
-	8400 700  8400 1550
-Wire Wire Line
-	8400 1550 8100 1550
-Wire Wire Line
-	8200 1650 8200 850
-Connection ~ 8200 1650
+	8200 800  8400 800
 $Comp
 L Device:Q_DUAL_NMOS_S1G1D2S2G2D1 Q2
@@
 $EndComp
 Wire Wire Line
-	8100 1250 8800 1250
-Wire Wire Line
 	8100 1350 10000 1350
-Wire Wire Line
-	8100 1450 8700 1450
 $Comp
 L power:VCC #PWR051
@@
 F 1 "430" V 9134 2600 50  0000 C CNN
 F 2 "Resistor_SMD:R_0402_1005Metric" V 9180 2600 50  0001 C CNN
-F 3 "https://datasheet.lcsc.com/szlcsc/1912111437_Viking-Tech-ARG02FTC4300_C284568.pdf" H 9250 2600 50  0001 C CNN
-F 4 "430 ±1% 1/16W 0402 High Precision & Low TCR SMD Resistors RoHS" V 9250 2600 50  0001 C CNN "description"
-F 5 "ARG02FTC4300" V 9250 2600 50  0001 C CNN "MPN"
+F 3 "https://www.tme.eu/Document/9e42ba54d36a9bd3dfa2901986ac022d/rezystor-smd.pdf" H 9250 2600 50  0001 C CNN
+F 4 "thick film; SMD; 0402; 430Ω; 63mW; ±1%; -55÷155°C" V 9250 2600 50  0001 C CNN "description"
+F 5 "0402WGF4300TCE" V 9250 2600 50  0001 C CNN "MPN"
 	1    9250 2600
 	-1   0    0    1
@@
 See note below.\nFor the NAND gate.
 Wire Wire Line
-	8800 1250 8800 3000
-Wire Wire Line
 	8800 3000 8950 3000
-Connection ~ 8800 1250
-Wire Wire Line
-	8800 1250 9850 1250
-Connection ~ 8700 1450
-Wire Wire Line
-	8700 1450 9800 1450
 Wire Wire Line
 	8700 3400 8950 3400
-Wire Wire Line
-	8700 1450 8700 3400
 Wire Wire Line
 	9250 2800 9750 2800
@@
 NoConn ~ 1900 4400
 NoConn ~ 1900 4200
-Wire Wire Line
-	8200 1650 8600 1650
 Text Notes 700  1400 0    50   ~ 0
 VBATOUT is BT1+ or USB VBUS.
@@
 $EndComp
 Text Notes 9950 1000 0    50   ~ 0
-When there is USB power, \nADC1 is disconnected.
+When there is USB power, \nXVCC is grounded.
 Text Notes 9950 800  0    50   ~ 0
-ADC1 point is intended for\nconnecting a microphone\nor other input to the ATtiny.
+XSIG1 and XSIG2 are intended for\nconnecting a microphone, buzzer\nor EEPROM or other addon boards.
 Text Notes 6750 4800 0    50   ~ 0
 Unused,\ngrounded.
@@
 Wire Wire Line
 	3200 1500 3800 1500
-Wire Wire Line
-	8600 1650 8600 800
 $Comp
 L power:VCC #PWR055
@@
 Wire Wire Line
 	5800 1500 5900 1500
-Text GLabel 8600 800  2    50   Input ~ 0
+Text GLabel 8650 650  2    50   Input ~ 0
 XSIG1
 $Comp
-L Connector:Conn_01x04_Female J1
+L Connector:Conn_01x06_Female J1
 U 1 1 5E48E7B6
 P 3800 6900
 F 0 "J1" H 3828 6830 50  0000 L CNN
-F 1 "THD0509-04CL-GF" H 3828 6785 50  0001 L CNN
-F 2 "chase-libs:THD050904CLGF" H 3800 6900 50  0001 C CNN
-F 3 "https://datasheet.lcsc.com/szlcsc/1811021341_THD-THD0509-04CL-GF_C283133.pdf" H 3800 6900 50  0001 C CNN
-F 4 "THD0509-04CL-GF" H 3800 6900 50  0001 C CNN "MPN"
-F 5 "FPC Contact,Top and Bottom 4 0.020\"（0.50mm） SMD,P=0.5mm FFC, FPC Connectors RoHS" H 3800 6900 50  0001 C CNN "Description"
+F 1 "FH12-6S-0.5SH(55)" H 3828 6785 50  0001 L CNN
+F 2 "Connector_FFC-FPC:Hirose_FH12-6S-0.5SH_1x06-1MP_P0.50mm_Horizontal" H 3800 6900 50  0001 C CNN
+F 3 "https://www.hirose.com/product/document?clcode=CL0586-0582-5-55&productname=FH12-6S-0.5SH(55)&series=FH12&documenttype=Catalog&lang=en&documentid=D31648_en" H 3800 6900 50  0001 C CNN
+F 4 "FH12-6S-0.5SH(55)" H 3800 6900 50  0001 C CNN "MPN"
+F 5 "FPC Contact 6pin SMD horizontal" H 3800 6900 50  0001 C CNN "Description"
 	1    3800 6900
 	1    0    0    -1
@@
 Wire Wire Line
 	3450 7100 3600 7100
-Text GLabel 3600 6800 0    50   Input ~ 0
+Text GLabel 3600 6700 0    50   Input ~ 0
 XSIG1
 Text GLabel 3600 6900 0    50   Input ~ 0
@@
 Wire Wire Line
 	1600 7050 1850 7050
+Wire Wire Line
+	8100 1550 8800 1550
+Wire Wire Line
+	8800 1550 8800 3000
+Wire Wire Line
+	8800 1550 9600 1550
+Wire Wire Line
+	9600 1550 9600 1450
+Wire Wire Line
+	9600 1450 9850 1450
+Connection ~ 8800 1550
+Connection ~ 9850 1450
+Wire Wire Line
+	8100 1650 8700 1650
+Wire Wire Line
+	9650 1650 9650 1550
+Wire Wire Line
+	9650 1550 9800 1550
+Connection ~ 9800 1550
+Wire Wire Line
+	8700 3400 8700 1650
+Connection ~ 8700 1650
+Wire Wire Line
+	8700 1650 9650 1650
+Wire Wire Line
+	8200 650  8550 650
+Wire Wire Line
+	8100 1450 8400 1450
+Wire Wire Line
+	8100 1250 8550 1250
+Connection ~ 8550 650
+Wire Wire Line
+	8550 650  8650 650
+Text GLabel 8200 800  0    50   Input ~ 0
+D+
+Wire Wire Line
+	8400 800  8400 1450
+Wire Wire Line
+	8550 650  8550 1250
+Text GLabel 8650 800  2    50   Input ~ 0
+XSIG2
+Wire Wire Line
+	8400 800  8650 800
+Connection ~ 8400 800
+Text GLabel 3600 6800 0    50   Input ~ 0
+XSIG2
+NoConn ~ 3600 7200
 $EndSCHEMATC

Commit message: Change TPS63000 variable to TPS63001 3.3V buck-boost.
TPS630001 is in stock now, can use it again. R73 and R74 are not
necessary now.

Change resistor brand for 71.5ohm resistors.

From VikingTech to UniRoyal which is cheaper.
Parts:
- removed R73: 1M, Resistor_SMD:R_0603_1608Metric, symbol Device:R
- removed R74: 178K, Resistor_SMD:R_0603_1608Metric, symbol Device:R
- R68, R69: MPN ARG02FTC71R5 -> 0402WGF715JTCE; description 71.5 ±1% 1/16W 0402 High Precision & Low TCR SMD Resistors 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 -> 71.5 ±1% 1/16W ±200ppm/℃ 0402 Chip Resistor - Surface Mount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
Connections:
- net VCC: now also U2.10 (FB)
Changed lines of the file:
@@
 F 1 "75.1" V 2334 5450 50  0000 C CNN
 F 2 "Resistor_SMD:R_0402_1005Metric" V 2380 5450 50  0001 C CNN
-F 3 "https://datasheet.lcsc.com/szlcsc/1810261110_Viking-Tech-ARG02FTC71R5_C284673.pdf" H 2450 5450 50  0001 C CNN
-F 4 "71.5 ±1% 1/16W 0402 High Precision & Low TCR SMD Resistors RoHS" V 2450 5450 50  0001 C CNN "description"
-F 5 "ARG02FTC71R5" V 2450 5450 50  0001 C CNN "MPN"
+F 3 "https://datasheet.lcsc.com/szlcsc/1810301125_UNI-ROYAL-Uniroyal-Elec-0402WGF715JTCE_C270584.pdf" H 2450 5450 50  0001 C CNN
+F 4 "71.5 ±1% 1/16W ±200ppm/℃ 0402 Chip Resistor - Surface Mount RoHS" V 2450 5450 50  0001 C CNN "description"
+F 5 "0402WGF715JTCE" V 2450 5450 50  0001 C CNN "MPN"
 	1    2450 5450
 	0    1    1    0
@@
 F 1 "75.1" V 2334 5750 50  0000 C CNN
 F 2 "Resistor_SMD:R_0402_1005Metric" V 2380 5750 50  0001 C CNN
-F 3 "https://datasheet.lcsc.com/szlcsc/1810261110_Viking-Tech-ARG02FTC71R5_C284673.pdf" H 2450 5750 50  0001 C CNN
-F 4 "71.5 ±1% 1/16W 0402 High Precision & Low TCR SMD Resistors RoHS" V 2450 5750 50  0001 C CNN "description"
-F 5 "ARG02FTC71R5" V 2450 5750 50  0001 C CNN "MPN"
+F 3 "https://datasheet.lcsc.com/szlcsc/1810301125_UNI-ROYAL-Uniroyal-Elec-0402WGF715JTCE_C270584.pdf" H 2450 5750 50  0001 C CNN
+F 4 "71.5 ±1% 1/16W ±200ppm/℃ 0402 Chip Resistor - Surface Mount RoHS" V 2450 5750 50  0001 C CNN "description"
+F 5 "0402WGF715JTCE" V 2450 5750 50  0001 C CNN "MPN"
 	1    2450 5750
 	0    1    1    0
@@
 Connection ~ 6000 2550
 Connection ~ 5800 2250
-$Comp
-L Device:R R73
-U 1 1 5E415EFC
-P 3200 1700
-F 0 "R73" V 2993 1700 50  0000 C CNN
-F 1 "1M" V 3084 1700 50  0000 C CNN
-F 2 "Resistor_SMD:R_0603_1608Metric" V 3130 1700 50  0001 C CNN
-F 3 "https://datasheet.lcsc.com/szlcsc/1811141225_Viking-Tech-AR03BTCX1004_C318138.pdf" H 3200 1700 50  0001 C CNN
-F 4 "1M ±0.1% 1/10W 0603 High Precision & Low TCR SMD Resistors RoHS" V 3200 1700 50  0001 C CNN "description"
-F 5 "AR03BTCX1004" V 3200 1700 50  0001 C CNN "MPN"
-	1    3200 1700
-	-1   0    0    1
-$EndComp
-$Comp
-L Device:R R74
-U 1 1 5E41640F
-P 3200 2100
-F 0 "R74" V 2993 2100 50  0000 C CNN
-F 1 "178K" V 3084 2100 50  0000 C CNN
-F 2 "Resistor_SMD:R_0603_1608Metric" V 3130 2100 50  0001 C CNN
-F 3 "https://datasheet.lcsc.com/szlcsc/1912111437_UNI-ROYAL-Uniroyal-Elec-TC0350B1783T5E_C425429.pdf" H 3200 2100 50  0001 C CNN
-F 4 "178K ±0.1% 1/6W ±50ppm℃ 0603 High Precision & Low TCR SMD Resistors RoHS" V 3200 2100 50  0001 C CNN "description"
-F 5 "TC0350B1783T5E" V 3200 2100 50  0001 C CNN "MPN"
-	1    3200 2100
-	-1   0    0    1
-$EndComp
-$Comp
-L power:GND #PWR054
-U 1 1 5E432DBA
-P 3200 2350
-F 0 "#PWR054" H 3200 2100 50  0001 C CNN
-F 1 "GND" H 3205 2177 50  0000 C CNN
-F 2 "" H 3200 2350 50  0001 C CNN
-F 3 "" H 3200 2350 50  0001 C CNN
-	1    3200 2350
-	1    0    0    -1
-$EndComp
-Wire Wire Line
-	3200 2350 3200 2250
-Wire Wire Line
-	3200 1850 3200 1900
 Wire Wire Line
 	3050 1500 3200 1500
-Wire Wire Line
-	3200 1900 3050 1900
-Wire Wire Line
-	3050 1700 3050 1900
-Connection ~ 3200 1900
-Wire Wire Line
-	3200 1900 3200 1950
 Connection ~ 3200 1500
 $Comp
@@
 	1    0    0    -1
 $EndComp
-Wire Wire Line
-	3200 1550 3200 1500
 Wire Wire Line
 	3600 2100 3600 2200
@@
 XSIG2
 NoConn ~ 3600 7200
+Wire Wire Line
+	3050 1700 3200 1700
+Wire Wire Line
+	3200 1500 3200 1700
 $EndSCHEMATC
